File: design/rotationdisplaymod/rotationdisplaymod.kicad_pcb (KiCad board)
At the start: 2 copper layers, 16 parts, among them J1 Power_Terminal, J2 Prog_Con_1, J3 Prog_Con_2, J4 LED_Con, J5 Joy_Con, J6 Motor_Terminal, Q1 BS250, Q2 2N7000, U1 ATtiny85-20PU, U2 L293D

Commit message: first production, kicad
Parts:
- removed the J3 at (125.7, 41.9)
- J2: value Prog_Con_1 -> Prog_Con; footprint Connector_PinHeader_2.00mm:PinHeader_1x03_P2.00mm_Vertical -> Connector_PinHeader_2.00mm:PinHeader_1x08_P2.00mm_Vertical
- moved D2 48.9 mm to (104.1, 61.0)
- moved R3 45.1 mm to (110.5, 61.0)
- moved D1 42.8 mm to (104.1, 54.6)
- moved J2 42.2 mm to (91.4, 71.1), turned to 90 degrees
- moved J3 39.3 mm to (133.3, 63.5)
- moved Q1 34.7 mm to (117.0, 55.3)
- moved Q2 34.7 mm to (117.0, 61.1)
- moved R2 31.3 mm to (110.5, 54.6)
- moved J4 28.7 mm to (133.3, 54.6)
- moved R1 22.0 mm to (125.7, 54.6), turned to 270 degrees
- moved U1 15.9 mm to (91.4, 57.1), turned to 0 degrees
- moved U2 12.0 mm to (104.1, 49.5)
- moved C1 11.7 mm to (99.1, 53.3), turned to 180 degrees
- moved J5 3.81 mm to (132.1, 48.3)
- renumbered J4 to J3, J5 to J4, J6 to J5
Connections:
- net Net-(D2-Pad2) renamed /NPin0
- net Net-(J5-Pad1) renamed /Pin3
- net Net-(J6-Pad1) renamed /Motor1
- net Net-(J6-Pad2) renamed /Motor2
- net Net-(U1-Pad3) renamed /Pin4
- D1 pad 2: Net-(D1-Pad2) -> /Pin0
- J2 pad 2: Net-(J2-Pad2) -> /VCC
- J2 pad 3: Net-(J2-Pad3) -> /GND
- J3 pad 1: Net-(J2-Pad3) -> /Pin1
- J3 pad 2: Net-(J2-Pad2) -> /Pin2
- Q1 pad 2: Net-(D1-Pad2) -> /Pin0
- Q2 pad 2: Net-(D1-Pad2) -> /Pin0
- U1 pad 1: Net-(J2-Pad1) -> /Reset
- U1 pad 5: Net-(D1-Pad2) -> /Pin0
- U1 pad 6: Net-(J2-Pad3) -> /Pin1
- U1 pad 7: Net-(J2-Pad2) -> /Pin2
- U2 pad 2: Net-(D1-Pad2) -> /Pin0
Routing:
- net /VCC: track 0.00 -> 98.8 mm
- net /Pin0: track 0.00 -> 50.9 mm
- net /Pin2: track 0.00 -> 48.8 mm
- net /Pin1: track 0.00 -> 48.8 mm
- net /Pin3: track 0.00 -> 44.4 mm
- net /Reset: track 0.00 -> 28.6 mm
- net /Motor2: track 0.00 -> 26.9 mm
- net /NPin0: track 0.00 -> 26.9 mm
- net /Motor1: track 0.00 -> 24.4 mm
- net /Pin4: track 0.00 -> 24.3 mm
- net Net-(D2-Pad1): track 0.00 -> 7.41 mm
- net Net-(D1-Pad1): track 0.00 -> 7.41 mm
- added copper zone on B.Cu, net /GND
- added copper zone on F.Cu, net /GND
Other:
- board outline added: 50.8 x 35.6 mm
- net class Default: clearance 0.2 -> 0.254; trace_width 0.25 -> 0.254
- net class VCC added: clearance 0.254, trace_width 0.762, via_dia 0.8, via_drill 0.4
- rule trace_clearance: 0.2 -> 0.254
- board text added: "Controller For Rotation Display Stands RGB Capable"
- board text added: "by BadGitZ"
