File: design/rotationdisplaymod/rotationdisplaymod.sch (KiCad schematic (older format))
At the start: 16 parts, among them J1 Power_Terminal, J2 Prog_Con_1, J3 Prog_Con_2, J4 LED_Con, J5 Joy_Con, J6 Motor_Terminal, Q1 BS250, Q2 2N7000, U1 ATtiny85-20PU, U2 L293D

Commit message: first production, kicad
Parts:
- removed J2: Prog_Con_1, Connector_PinHeader_2.00mm:PinHeader_1x03_P2.00mm_Vertical, symbol Connector:Conn_01x03_Male
- removed J3: Prog_Con_2, Connector_PinHeader_2.00mm:PinHeader_1x03_P2.00mm_Vertical, symbol Connector:Conn_01x03_Male
- added J2: Prog_Con, Connector_PinHeader_2.00mm:PinHeader_1x08_P2.00mm_Vertical, symbol Connector:Conn_01x08_Male
- renumbered J4 to J3, J5 to J4, J6 to J5
Connections:
- net GND: now also J2.3 (Pin_3)
- net VCC: now also J2.2 (Pin_2)
- net Reset: now reaches U1.1 (~RESET~/PB5)
- net Reset: now also J2.6 (Pin_6)
- net Pin3: now reaches J4.1 (Pin_1), R1.1, U1.2 (XTAL1/PB3)
- net Pin4: now reaches U1.3 (XTAL2/PB4), U2.1 (EN1,2)
- net Pin0: now reaches D1.2 (A), Q1.2 (G), Q2.2 (G), U1.5 (AREF/PB0), U2.2 (1A)
- net Pin0: now also J2.7 (Pin_7)
- net Pin1: now reaches J3.1 (Pin_1), U1.6 (PB1)
- net Pin1: now also J2.4 (Pin_4)
- net Pin2: now reaches J3.2 (Pin_2), U1.7 (PB2)
- net Pin2: now also J2.5 (Pin_5)
- net Motor1: now reaches J5.1 (Pin_1), U2.3 (1Y)
- net Motor2: now reaches J5.2 (Pin_2), U2.6 (2Y)
- net NPin0: now reaches D2.2 (A), Q1.3 (S), Q2.3 (D), U2.7 (2A)
- no-connect marks 6 -> 7
Changed lines of the file:
@@
 Sheet 1 1
 Title "Rotation Display Controller"
-Date "2020-08-13"
+Date "2020-09-26"
 Rev "v01"
 Comp "BadGitZ"
@@
 	2150 2750 2150 2400
 Wire Wire Line
-	2150 2400 2800 2400
-Wire Wire Line
-	3500 3600 4300 3600
+	2150 2400 2600 2400
 Connection ~ 3500 3600
 Wire Wire Line
@@
 	5400 2900 5400 2800
 $Comp
-L Connector:Screw_Terminal_01x02 J6
+L Connector:Screw_Terminal_01x02 J5
 U 1 1 5F373F07
 P 7000 2850
-F 0 "J6" H 7080 2842 50  0000 L CNN
+F 0 "J5" H 7080 2842 50  0000 L CNN
 F 1 "Motor_Terminal" H 7080 2751 50  0000 L CNN
 F 2 "TerminalBlock:TerminalBlock_bornier-2_P5.08mm" H 7000 2850 50  0001 C CNN
@@
 	6000 2050 6000 2400
 Connection ~ 5800 2050
-$Comp
-L Connector:Conn_01x03_Male J2
-U 1 1 5F3EF034
-P 3300 4300
-F 0 "J2" H 3400 4450 50  0000 R CNN
-F 1 "Prog_Con_1" H 3750 4550 50  0000 R CNN
-F 2 "Connector_PinHeader_2.00mm:PinHeader_1x03_P2.00mm_Vertical" H 3300 4300 50  0001 C CNN
-F 3 "~" H 3300 4300 50  0001 C CNN
-	1    3300 4300
-	-1   0    0    1
-$EndComp
-$Comp
-L Connector:Conn_01x03_Male J3
-U 1 1 5F3F083C
-P 3350 4300
-F 0 "J3" H 3400 4150 50  0000 C CNN
-F 1 "Prog_Con_2" H 3600 4050 50  0000 C CNN
-F 2 "Connector_PinHeader_2.00mm:PinHeader_1x03_P2.00mm_Vertical" H 3350 4300 50  0001 C CNN
-F 3 "~" H 3350 4300 50  0001 C CNN
-	1    3350 4300
-	1    0    0    -1
-$EndComp
 Wire Wire Line
 	4100 3200 4100 3700
 Wire Wire Line
-	4100 3700 2850 3700
-Wire Wire Line
-	2850 3700 2850 4400
-Wire Wire Line
-	2850 4400 3100 4400
+	4100 3700 3450 3700
 Wire Wire Line
 	4100 2900 4150 2900
@@
 	4150 2900 4150 3750
 Wire Wire Line
-	4150 3750 2900 3750
-Wire Wire Line
-	2900 3750 2900 4300
-Wire Wire Line
-	2900 4300 3100 4300
-Wire Wire Line
-	2950 3800 2950 4200
-Wire Wire Line
-	2950 4200 3100 4200
-NoConn ~ 3550 4200
+	4150 3750 3350 3750
 Wire Wire Line
 	4100 3100 4850 3100
 Wire Wire Line
-	4200 3800 2950 3800
+	4200 3800 3250 3800
 Wire Wire Line
 	4100 2700 4250 2700
@@
 Wire Wire Line
 	4250 2900 4250 3850
-Wire Wire Line
-	4250 3850 3650 3850
-Wire Wire Line
-	3650 3850 3650 4300
-Wire Wire Line
-	3650 4300 3550 4300
 Connection ~ 4250 2900
-Wire Wire Line
-	4300 3600 4300 3900
-Wire Wire Line
-	4300 3900 3700 3900
-Wire Wire Line
-	3700 3900 3700 4400
-Wire Wire Line
-	3700 4400 3550 4400
-Connection ~ 4300 3600
-Wire Wire Line
-	4300 3600 4450 3600
-$Comp
-L Connector:Conn_01x02_Male J5
+$Comp
+L Connector:Conn_01x02_Male J4
 U 1 1 5F405687
 P 4700 1450
-F 0 "J5" H 4672 1332 50  0000 R CNN
+F 0 "J4" H 4672 1332 50  0000 R CNN
 F 1 "Joy_Con" H 4672 1423 50  0000 R CNN
 F 2 "Connector_PinHeader_2.00mm:PinHeader_1x02_P2.00mm_Vertical" H 4700 1450 50  0001 C CNN
@@
 Connection ~ 4450 3000
 $Comp
-L Connector:Conn_01x04_Male J4
+L Connector:Conn_01x04_Male J3
 U 1 1 5F40C008
 P 4050 1450
-F 0 "J4" V 4112 1594 50  0000 L CNN
+F 0 "J3" V 4112 1594 50  0000 L CNN
 F 1 "LED_Con" V 4203 1594 50  0000 L CNN
 F 2 "Connector_PinHeader_2.00mm:PinHeader_1x04_P2.00mm_Vertical" H 4050 1450 50  0001 C CNN
@@
 Connection ~ 2900 3600
 Wire Wire Line
-	2900 3600 3500 3600
+	2900 3600 3150 3600
 Wire Wire Line
 	4150 2900 4150 2250
@@
 	4200 2200 4200 2800
 Connection ~ 4200 2800
+$Comp
+L Connector:Conn_01x08_Male J2
+U 1 1 5F6FCD72
+P 3250 4800
+F 0 "J2" V 3177 4728 50  0000 C CNN
+F 1 "Prog_Con" V 3086 4728 50  0000 C CNN
+F 2 "Connector_PinHeader_2.00mm:PinHeader_1x08_P2.00mm_Vertical" H 3250 4800 50  0001 C CNN
+F 3 "~" H 3250 4800 50  0001 C CNN
+	1    3250 4800
+	0    -1   -1   0
+$EndComp
+Wire Wire Line
+	2600 2400 2600 4550
+Wire Wire Line
+	2600 4550 3050 4550
+Wire Wire Line
+	3050 4550 3050 4600
+Connection ~ 2600 2400
+Wire Wire Line
+	2600 2400 2800 2400
+NoConn ~ 2950 4600
+Wire Wire Line
+	3250 3800 3250 4600
+Wire Wire Line
+	3350 4600 3350 3750
+Wire Wire Line
+	3450 4600 3450 3700
+Wire Wire Line
+	3550 3850 3550 4600
+Wire Wire Line
+	3550 3850 4250 3850
+Connection ~ 3150 3600
+Wire Wire Line
+	3150 3600 3500 3600
+Wire Wire Line
+	3150 3600 3150 4600
+Wire Wire Line
+	3500 3600 4450 3600
+NoConn ~ 3650 4600
+Text Label 3700 3700 0    50   ~ 0
+Reset
+Text Label 4300 2500 0    50   ~ 0
+Pin0
+Text Label 4150 1900 0    50   ~ 0
+Pin1
+Text Label 4050 2000 0    50   ~ 0
+Pin2
+Text Label 4700 1850 0    50   ~ 0
+Pin3
+Text Label 4700 3100 0    50   ~ 0
+Pin4
+Text Label 5050 2600 0    50   ~ 0
+NPin0
+Text Label 6550 2850 0    50   ~ 0
+Motor1
+Text Label 6550 2950 0    50   ~ 0
+Motor2
 $EndSCHEMATC
